File: PiZero-RAK.sch (EAGLE design)
At the start: 36 parts, among them IC1 PCF8523, J1 CON_HEADER_1X05-PTH, J11 CON_HEADER_1X06-PTH, J2 CONN_20X2HLE, J3 CON_HEADER_1X05-PTH, J4 CON_HEADER_1X05-PTH, Q1 CJ2302, X1 SPTAF_23.5, X2 SPTAF_25.0MM, Y1 32.768KHz

Commit message: My version
Change 10cm Max
Parts:
- removed X2: SPTAF_25.0MM, _c2h:SPTAF_25.0MM
- added IN: (no value), con-phoenix-254:MPT3
- R2: device _c2h:RESISTORPTH-1/4W -> _c2h:RESISTORAXIAL-0.3
- X1: value SPTAF_23.5 -> (none); device _c2h:SPTAF_23.5 -> con-phoenix-254:MPT2
Connections:
- net 3V3: no longer X1-2.2
- net GND: now also IN-1.1, IN-2.1; no longer X2-1.1, X2-1.2
- net GPIO17: no longer X1-1.2
- net VIN: now also IN-3.1; no longer X2-2.1, X2-2.2
